Commit message: Added Plugins

File: urdf/inferno_simulation.urdf (robot description, URDF)
Before this commit: robot inferno_simulation, 8 links, 7 joints
Links:
- link base_link: mass 0.418054450091855 -> 1
Joints:
- joint lidar_joint: origin xyz=-0.18876 -0.15318 0.011436 rpy=1.5708 0 3.1416 -> xyz=-0.18876 -0.15318 0.011436 rpy=0 0 0
